File: PCB/Sensorbox.kicad_sch (KiCad schematic)
At the start: 28 parts, among them J101 Prog_Pin, J102 Barrel_Jack_MountingPin, SW101 Reset, SW102 Reset, U101 ESP-12F, U102 LM7805_TO220, U103 L79L05_TO92

Commit message: added drill files
Parts:
- removed SB103: ~, symbol thu_sensoren_tht:DHT11_Board
- added H101, H102, H103, H104: MountingHole, MountingHole:MountingHole_3.2mm_M3, symbol Mechanical:MountingHole
- added JP101: Power 5/12V, Jumper:SolderJumper-3_P1.3mm_Open_RoundedPad1.0x1.5mm_NumberLabels, symbol Jumper:SolderJumper_3_Bridged123
- added SB103: DHT22_Board, sensoren-tht:DHT22-horizontal, symbol thu_sensoren_tht:DHT22_Board
- SB101: footprint (none) -> sensoren-tht:RCWL-0516
- SB102: footprint (none) -> sensoren-tht:BMP180
- SB104: footprint (none) -> sensoren-tht:SR602_Board
- SB105: footprint (none) -> sensoren-tht:MQ-2
- SW101: footprint (none) -> switch-tht:Button
- SW102: value Reset -> Prog; footprint (none) -> switch-tht:Button
- U102: footprint Package_TO_SOT_SMD:SOT-23-5_HandSoldering -> Package_TO_SOT_THT:TO-220-3_Vertical
- UB101: footprint (none) -> sensoren-tht:ADC1115_Board
Connections:
- net +5V: now also JP101.1 (A), SB103.1 (VIN); no longer SB101.2 (VIN)
- net GND: now also J102.3 (MountPin), SB103.3 (GND); no longer J102.MP (MountPin)
- net VCC: now also JP101.3 (B)
- net Data_DHT11 renamed Data_DHT22
- net Data_DHT22: now also SB103.2 (OUT)
- new net: JP101.2 (C), SB101.2 (VIN)
Other:
- moved on the sheet: J102
